File: kicad/5uH_LISN.kicad_pcb (KiCad board)
At the start: 2 copper layers, 100 x 50 mm, 37 parts, among them J1 BANANA_CONN, J2 BANANA_CONN, J3 BANANA_CONN, J4 BANANA_CONN

Commit message: Replaced C2 with C2220 for higher voltage rating.  Schematic symbol for C2 no longer polarized.  More via stitching.
Parts:
- C2: footprint 5uH_LISN:PANASONIC_B -> Capacitor_SMD:C_2220_5650Metric
- moved C2 7.00 mm to (185.0, 105.0)
- moved C1 5.00 mm to (180.0, 105.0)
Routing:
- net GND: vias 33 -> 58
Changed lines of the file:
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@@
     (thickness 1.6)
     (drawings 19)
-    (tracks 74)
+    (tracks 99)
     (zones 0)
     (modules 37)
@@
     (47 F.CrtYd user)
     (48 B.Fab user)
-    (49 F.Fab user)
+    (49 F.Fab user hide)
   )
   (setup
@@
     (add_net "Net-(L4-Pad2)")
   )
+  (module Capacitor_SMD:C_2220_5650Metric (layer Top)
+    (at 185 105 90)
+    (descr "Capacitor SMD 2220 (5650 Metric), square (rectangular) end terminal, IPC_7351 nominal, (Body size from: http://datasheets.avx.com/AVX-HV_MLCC.pdf), generated with kicad-footprint-generator")
+    (tags capacitor)
+    (attr smd)
+    (fp_text reference C2 (at -2 3.5 270) (layer F.SilkS)
+      (effects (font (size 0.9652 0.9652) (thickness 0.077216)) (justify right top))
+    )
+    (fp_text value 22u (at -2.15 3.275 90) (layer F.Fab)
+      (effects (font (size 0.9652 0.9652) (thickness 0.077216)) (justify left bottom))
+    )
+    (fp_text user %R (at 0 0 90) (layer F.Fab)
+      (effects (font (size 1 1) (thickness 0.15)))
+    )
+    (fp_line (start 3.7 2.95) (end -3.7 2.95) (layer F.CrtYd) (width 0.05))
+    (fp_line (start 3.7 -2.95) (end 3.7 2.95) (layer F.CrtYd) (width 0.05))
+    (fp_line (start -3.7 -2.95) (end 3.7 -2.95) (layer F.CrtYd) (width 0.05))
+    (fp_line (start -3.7 2.95) (end -3.7 -2.95) (layer F.CrtYd) (width 0.05))
+    (fp_line (start -1.415748 2.61) (end 1.415748 2.61) (layer F.SilkS) (width 0.12))
+    (fp_line (start -1.415748 -2.61) (end 1.415748 -2.61) (layer F.SilkS) (width 0.12))
+    (fp_line (start 2.85 2.5) (end -2.85 2.5) (layer F.Fab) (width 0.1))
+    (fp_line (start 2.85 -2.5) (end 2.85 2.5) (layer F.Fab) (width 0.1))
+    (fp_line (start -2.85 -2.5) (end 2.85 -2.5) (layer F.Fab) (width 0.1))
+    (fp_line (start -2.85 2.5) (end -2.85 -2.5) (layer F.Fab) (width 0.1))
+    (pad 2 smd roundrect (at 2.55 0 90) (size 1.8 5.4) (layers Top F.Paste F.Mask) (roundrect_rratio 0.138889))
+    (pad 1 smd roundrect (at -2.55 0 90) (size 1.8 5.4) (layers Top F.Paste F.Mask) (roundrect_rratio 0.138889))
+    (model ${KISYS3DMOD}/Capacitor_SMD.3dshapes/C_2220_5650Metric.wrl
+      (at (xyz 0 0 0))
+      (scale (xyz 1 1 1))
+      (rotate (xyz 0 0 0))
+    )
+  )
   (module 5uH_LISN:C1210 (layer Top)
-    (at 185 105 270)
+    (at 180 105 270)
     (descr <b>CAPACITOR</b>)
-    (fp_text reference C1 (at -1.905 -1.905) (layer F.SilkS)
+    (fp_text reference C1 (at 2 2 90) (layer F.SilkS)
       (effects (font (size 0.9652 0.9652) (thickness 0.077216)) (justify left bottom))
     )
@@
     (pad 1 smd rect (at -1.4 0 270) (size 1.6 2.7) (layers Top F.Paste F.Mask)
       (net 3 "Net-(C1-Pad1)") (solder_mask_margin 0.1016))
-  )
-  (module 5uH_LISN:PANASONIC_B (layer Top)
-    (at 178.0011 105.0036 90)
-    (descr "<b>Panasonic Aluminium Electrolytic Capacitor VS-Serie Package B</b>")
-    (fp_text reference C2 (at -2.15 -2.3) (layer F.SilkS)
-      (effects (font (size 0.9652 0.9652) (thickness 0.077216)) (justify right top))
-    )
-    (fp_text value 22u (at -2.15 3.275 90) (layer F.Fab)
-      (effects (font (size 0.9652 0.9652) (thickness 0.077216)) (justify left bottom))
-    )
-    (fp_poly (pts (xy -1.25 -1.45) (xy -1.7 -0.85) (xy -1.85 -0.35) (xy -1.85 0.4)
-      (xy -1.7 0.85) (xy -1.25 1.4) (xy -1.25 -1.4)) (layer F.Fab) (width 0))
-    (fp_poly (pts (xy 1.9 0.35) (xy 2.3 0.35) (xy 2.3 -0.35) (xy 1.9 -0.35)) (layer F.Fab) (width 0))
-    (fp_poly (pts (xy -2.3 0.35) (xy -1.85 0.35) (xy -1.85 -0.35) (xy -2.3 -0.35)) (layer F.Fab) (width 0))
-    (fp_circle (center 0 0) (end 1.95 0) (layer F.Fab) (width 0.1016))
-    (fp_line (start -1.2 -1.5) (end -1.2 1.5) (layer F.Fab) (width 0.1016))
-    (fp_line (start -2.1 2.1) (end -2.1 0.85) (layer F.SilkS) (width 0.1016))
-    (fp_line (start 1 2.1) (end -2.1 2.1) (layer F.SilkS) (width 0.1016))
-    (fp_line (start 2.1 1) (end 1 2.1) (layer F.SilkS) (width 0.1016))
-    (fp_line (start 1 -2.1) (end 2.1 -1) (layer F.SilkS) (width 0.1016))
-    (fp_line (start -2.1 -2.1) (end 1 -2.1) (layer F.SilkS) (width 0.1016))
-    (fp_line (start -2.1 -0.85) (end -2.1 -2.1) (layer F.SilkS) (width 0.1016))
-    (fp_arc (start 0 0) (end -1.75 0.85) (angle -128.186984) (layer F.SilkS) (width 0.1016))
-    (fp_arc (start 0 0) (end -1.75 -0.85) (angle 128.186984) (layer F.SilkS) (width 0.1016))
-    (fp_line (start -2.1 2.1) (end -2.1 -2.1) (layer F.Fab) (width 0.1016))
-    (fp_line (start 1 2.1) (end -2.1 2.1) (layer F.Fab) (width 0.1016))
-    (fp_line (start 2.1 1) (end 1 2.1) (layer F.Fab) (width 0.1016))
-    (fp_line (start 2.1 -1) (end 2.1 1) (layer F.Fab) (width 0.1016))
-    (fp_line (start 1 -2.1) (end 2.1 -1) (layer F.Fab) (width 0.1016))
-    (fp_line (start -2.1 -2.1) (end 1 -2.1) (layer F.Fab) (width 0.1016))
-    (pad + smd rect (at 1.6 0 90) (size 2.2 1.4) (layers Top F.Paste F.Mask)
-      (net 3 "Net-(C1-Pad1)") (solder_mask_margin 0.1016))
-    (pad - smd rect (at -1.6 0 90) (size 2.2 1.4) (layers Top F.Paste F.Mask)
-      (net 1 GND) (solder_mask_margin 0.1016))
   )
   (module 5uH_LISN:C1206 (layer Top)
@@
   )
   (gr_text + (at 195 97) (layer B.SilkS)
-    (effects (font (size 5 5) (thickness 0.4)) (justify bottom mirror))
+    (effects (font (size 4 4) (thickness 0.4)) (justify bottom mirror))
   )
   (gr_text - (at 195 117) (layer B.SilkS)
@@
   (via (at 165 108) (size 0.8) (drill 0.4) (layers Top Bottom) (net 1))
   (via (at 180 108) (size 0.8) (drill 0.4) (layers Top Bottom) (net 1))
+  (via (at 180 123) (size 0.8) (drill 0.4) (layers Top Bottom) (net 1))
+  (via (at 185.1 123) (size 0.8) (drill 0.4) (layers Top Bottom) (net 1))
   (via (at 175 107.9) (size 0.8) (drill 0.4) (layers Top Bottom) (net 1))
-  (via (at 188 108) (size 0.8) (drill 0.4) (layers Top Bottom) (net 1))
-  (via (at 184 108) (size 0.8) (drill 0.4) (layers Top Bottom) (net 1))
+  (via (at 190 108) (size 0.8) (drill 0.4) (layers Top Bottom) (net 1))
+  (via (at 195 108) (size 0.8) (drill 0.4) (layers Top Bottom) (net 1))
+  (via (at 170 123) (size 0.8) (drill 0.4) (layers Top Bottom) (net 1))
+  (via (at 135 123) (size 0.8) (drill 0.4) (layers Top Bottom) (net 1))
+  (via (at 155 123) (size 0.8) (drill 0.4) (layers Top Bottom) (net 1))
+  (via (at 120 123) (size 0.8) (drill 0.4) (layers Top Bottom) (net 1))
+  (via (at 160 123) (size 0.8) (drill 0.4) (layers Top Bottom) (net 1))
+  (via (at 140 123) (size 0.8) (drill 0.4) (layers Top Bottom) (net 1))
+  (via (at 145 123) (size 0.8) (drill 0.4) (layers Top Bottom) (net 1))
+  (via (at 130 123) (size 0.8) (drill 0.4) (layers Top Bottom) (net 1))
+  (via (at 175 122.9) (size 0.8) (drill 0.4) (layers Top Bottom) (net 1))
+  (via (at 125 123) (size 0.8) (drill 0.4) (layers Top Bottom) (net 1))
+  (via (at 115 123) (size 0.8) (drill 0.4) (layers Top Bottom) (net 1))
+  (via (at 150 123) (size 0.8) (drill 0.4) (layers Top Bottom) (net 1))
+  (via (at 165 123) (size 0.8) (drill 0.4) (layers Top Bottom) (net 1))
+  (via (at 105 113) (size 0.8) (drill 0.4) (layers Top Bottom) (net 1))
+  (via (at 105 103) (size 0.8) (drill 0.4) (layers Top Bottom) (net 1))
+  (via (at 105 98) (size 0.8) (drill 0.4) (layers Top Bottom) (net 1))
+  (via (at 105 93) (size 0.8) (drill 0.4) (layers Top Bottom) (net 1))
+  (via (at 105 118) (size 0.8) (drill 0.4) (layers Top Bottom) (net 1))
+  (via (at 195 113) (size 0.8) (drill 0.4) (layers Top Bottom) (net 1))
+  (via (at 195 118) (size 0.8) (drill 0.4) (layers Top Bottom) (net 1))
+  (via (at 195 103) (size 0.8) (drill 0.4) (layers Top Bottom) (net 1))
+  (via (at 195 98) (size 0.8) (drill 0.4) (layers Top Bottom) (net 1))
+  (via (at 195 93) (size 0.8) (drill 0.4) (layers Top Bottom) (net 1))
   (segment (start 162.45 95) (end 167.55 95) (width 3) (layer Top) (net 2))
   (segment (start 172.45 95) (end 185 95) (width 3) (layer Top) (net 3))
