File: kicad/5uH_LISN.sch (KiCad schematic (older format))
At the start: 37 parts, among them J1 BANANA_CONN, J2 BANANA_CONN, J3 BANANA_CONN, J4 BANANA_CONN

Commit message: Replaced C2 with C2220 for higher voltage rating.  Schematic symbol for C2 no longer polarized.  More via stitching.
Parts:
- C2: footprint 5uH_LISN:PANASONIC_B -> Capacitor_SMD:C_2220_5650Metric; symbol 5uH_LISN-eagle-import:CPOL-EUB -> 5uH_LISN-eagle-import:C-EUC1210
Connections:
- net GND: now also C2.2; no longer C2.-
- net at C1.1, J1.P$1 (1), L1.1: now also C2.1; no longer C2.+
Changed lines of the file:
@@
 EESchema Schematic File Version 4
+LIBS:5uH_LISN-cache
 EELAYER 29 0
 EELAYER END
@@
 $EndComp
 $Comp
-L 5uH_LISN-eagle-import:CPOL-EUB C2
+L 5uH_LISN-eagle-import:C-EUC1210 C2
 U 1 0 544A10D139FF0AA9
 P 5000 1600
 F 0 "C2" H 5045 1619 59  0000 L BNN
 F 1 "22u" H 5045 1419 59  0000 L BNN
-F 2 "5uH_LISN:PANASONIC_B" H 5000 1600 50  0001 C CNN
+F 2 "Capacitor_SMD:C_2220_5650Metric" H 5000 1600 50  0001 C CNN
 F 3 "" H 5000 1600 50  0001 C CNN
 	1    5000 1600
